File: HW/rev_D/rev_D.sch (EAGLE design)
At the start: 38 parts, among them CN1 HEADER_1X4_, CN2 HEADER_1X5, Q1 BSS138, Q2 BSS138, Q3 BSS138, Q4 BSS138, Q5 BSS138, U3 AP2112K-3.3

Commit message: Files clean up & README update
Parts:
- removed R13: 10K, rcl:R-EU_R0805
- added C2: 10uF, rcl:C-EUC0805
- added R20, R21, R22: 10K, rcl:R-EU_R0805
- added SD_CARD: MICRO_SD_CARD_, dronecz:MICRO_SD_CARD_
- added SJ1: (no value), microbuilder:SOLDERJUMPER_2WAY0805
- CN1: value HEADER_1X4_ -> HEADER_1X4__; device dronecz:HEADER_1X4_ -> dronecz:HEADER_1X4__
Connections:
- removed net N$5: R13.1, U$1.IO18
- new net IO12: SJ1.3, U$1.IO12
- new net IO18: R21.1, SD_CARD.CLK, U$1.IO18
- new net IO19: R22.1, SD_CARD.DAT0, U$1.IO19
- new net N$1: LED1.C, SJ1.2
- net 3V3: now also C2.1, R20.2, R21.2, R22.2, SD_CARD.VCC
- net GND: now also C2.2, SD_CARD.GND, SD_CARD.VSS
- net IO22: now also SD_CARD.CD/DAT3
- net IO23: now also R20.1, SD_CARD.CMD, SJ1.1; no longer LED1.C
- net PRINTER_RESET: no longer R13.2
Other:
- note added: "uSD card"
- moved on the sheet: LED1, LED2, R17, R18
